File: PCB/Timerbox.sch (KiCad schematic (older format))
At the start: 29 parts, among them CON1 AVR-ISP-6, IC1 ATTINY4313-P, K1 ROT, P1 CON, P2 BTN1, P4 RST, P5 BTN0, Q1 2N3904, U1 78L05, U2 LM7812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

Commit message: New PCB
Parts:
- removed D2, D?: LED, ~, symbol LED
- removed K1: ROT, symbol CONN_3
- removed P?: CONN_14, symbol CONN_14
- removed R7, R?: 1k, ~, symbol R
- added P3: BTN2, symbol CONN_2
- added P6, P7: BTN3, symbol CONN_2
- added P8: BTN4, symbol CONN_2
- gave numbers to parts that had none: 1
Connections:
- net GND: now also P3.2 (PM), P6.2 (PM), P7.2 (PM), P8.2 (PM)
- net BTN0: now reaches IC1.12 ((AIN0/PCINT0)PB0), P2.1 (P1)
- net BTN1: now reaches IC1.13 ((AIN1/PCINT1)PB1), P5.1 (P1)
- net BTN5: now reaches IC1.9 ((PCINT16/OC0B/T1)PD5)
- net BTN5: now also P8.1 (P1)
- net ROT0 renamed BTN2
- net BTN2: now also P3.1 (P1)
- net ROT1 renamed BTN3
- net BTN3: now also P6.1 (P1)
- net SCK renamed BTN4
- net BTN4: now also P7.1 (P1)

Commit message: Changed contrast pot
Connections:
- net +5V: now also RV1.1
- net GND: now also RV1.3; no longer RV1.2
- net at LCD1.3 (CON): now also RV1.2; no longer RV1.1
- no-connect marks 2 -> 1
Changed lines of the file:
@@
 LIBS:g5v2
 LIBS:srd48
-LIBS:Timerbox-cache
 EELAYER 27 0
 EELAYER END
@@
 Sheet 1 1
 Title "Temperature sensor board"
-Date "2 dec 2014"
+Date "3 may 2015"
 Rev "0.1"
 Comp "Hackoteket"
@@
 	0    -1   -1   0
 $EndComp
+Text Label 5925 3650 0    60   ~ 0
+BTN0
+Text Label 6125 4500 2    60   ~ 0
+BTN0
+Text Label 6125 4600 0    60   ~ 0
+BTN1
+Text Label 6500 3650 0    60   ~ 0
+BTN1
+$Comp
+L CONN_2 P3
+U 1 1 547E3875
+P 7450 2875
+F 0 "P3" V 7400 2875 40  0000 C CNN
+F 1 "BTN2" V 7500 2875 40  0000 C CNN
+F 2 "" H 7450 2875 60  0000 C CNN
+F 3 "" H 7450 2875 60  0000 C CNN
+	1    7450 2875
+	0    -1   -1   0
+$EndComp
+$Comp
+L CONN_2 P6
+U 1 1 547E387B
+P 7900 2875
+F 0 "P6" V 7850 2875 40  0000 C CNN
+F 1 "BTN3" V 7950 2875 40  0000 C CNN
+F 2 "" H 7900 2875 60  0000 C CNN
+F 3 "" H 7900 2875 60  0000 C CNN
+	1    7900 2875
+	0    -1   -1   0
+$EndComp
+Text Label 7125 3450 0    60   ~ 0
+BTN2
+Text Label 7600 3450 0    60   ~ 0
+BTN3
+Text Label 6200 5200 0    60   ~ 0
+BTN4
+$Comp
+L CONN_2 P7
+U 1 1 547E3C34
+P 8350 2875
+F 0 "P7" V 8300 2875 40  0000 C CNN
+F 1 "BTN3" V 8400 2875 40  0000 C CNN
+F 2 "" H 8350 2875 60  0000 C CNN
+F 3 "" H 8350 2875 60  0000 C CNN
+	1    8350 2875
+	0    -1   -1   0
+$EndComp
+Text Label 8025 3400 0    60   ~ 0
+BTN4
+Text Label 7200 5875 2    60   ~ 0
+RL2
+Text Label 6125 5900 0    60   ~ 0
+BTN5
+$Comp
+L CONN_2 P8
+U 1 1 547E4433
+P 8725 2875
+F 0 "P8" V 8675 2875 40  0000 C CNN
+F 1 "BTN4" V 8775 2875 40  0000 C CNN
+F 2 "" H 8725 2875 60  0000 C CNN
+F 3 "" H 8725 2875 60  0000 C CNN
+	1    8725 2875
+	0    -1   -1   0
+$EndComp
+Text Label 8725 3600 0    60   ~ 0
+BTN5
 $Comp
 L POT RV1
@@
 	0    -1   1    0
 $EndComp
-NoConn ~ 9475 6575
-Text Label 5925 3650 0    60   ~ 0
-BTN0
-Text Label 6125 4500 2    60   ~ 0
-BTN0
-Text Label 6125 4600 0    60   ~ 0
-BTN1
-Text Label 6500 3650 0    60   ~ 0
-BTN1
-$Comp
-L CONN_2 P3
-U 1 1 547E3875
-P 7450 2875
-F 0 "P3" V 7400 2875 40  0000 C CNN
-F 1 "BTN2" V 7500 2875 40  0000 C CNN
-F 2 "" H 7450 2875 60  0000 C CNN
-F 3 "" H 7450 2875 60  0000 C CNN
-	1    7450 2875
-	0    -1   -1   0
-$EndComp
-$Comp
-L CONN_2 P6
-U 1 1 547E387B
-P 7900 2875
-F 0 "P6" V 7850 2875 40  0000 C CNN
-F 1 "BTN3" V 7950 2875 40  0000 C CNN
-F 2 "" H 7900 2875 60  0000 C CNN
-F 3 "" H 7900 2875 60  0000 C CNN
-	1    7900 2875
-	0    -1   -1   0
-$EndComp
-Text Label 7125 3450 0    60   ~ 0
-BTN2
-Text Label 7600 3450 0    60   ~ 0
-BTN3
-Text Label 6200 5200 0    60   ~ 0
-BTN4
-$Comp
-L CONN_2 P7
-U 1 1 547E3C34
-P 8350 2875
-F 0 "P7" V 8300 2875 40  0000 C CNN
-F 1 "BTN3" V 8400 2875 40  0000 C CNN
-F 2 "" H 8350 2875 60  0000 C CNN
-F 3 "" H 8350 2875 60  0000 C CNN
-	1    8350 2875
-	0    -1   -1   0
-$EndComp
-Text Label 8025 3400 0    60   ~ 0
-BTN4
-Text Label 7200 5875 2    60   ~ 0
-RL2
-Text Label 6125 5900 0    60   ~ 0
-BTN5
-$Comp
-L CONN_2 P8
-U 1 1 547E4433
-P 8725 2875
-F 0 "P8" V 8675 2875 40  0000 C CNN
-F 1 "BTN4" V 8775 2875 40  0000 C CNN
-F 2 "" H 8725 2875 60  0000 C CNN
-F 3 "" H 8725 2875 60  0000 C CNN
-	1    8725 2875
-	0    -1   -1   0
-$EndComp
 Wire Wire Line
 	2500 4600 3050 4600
@@
 	9650 6100 9650 6125
 Wire Wire Line
-	9650 6125 10050 6125
-Wire Wire Line
-	10050 6025 9725 6025
-Wire Wire Line
-	9725 6025 9725 5925
-Wire Wire Line
-	9725 5925 9475 5925
-Wire Wire Line
-	9475 6625 9475 6775
+	9525 6125 10050 6125
 Wire Wire Line
 	4400 2850 4400 2600
@@
 	4125 3250 3800 3250
 Wire Wire Line
-	9475 5925 9475 6075
-Wire Wire Line
-	9475 6625 9325 6625
-Wire Wire Line
-	9325 6625 9325 6325
-Wire Wire Line
 	5900 5350 5900 5200
 Connection ~ 5900 5200
@@
 Wire Wire Line
 	8625 3600 8725 3600
-Text Label 8725 3600 0    60   ~ 0
-BTN5
 Wire Wire Line
 	8825 3225 8825 3375
@@
 Wire Wire Line
 	9075 3750 8000 3750
+Wire Wire Line
+	9475 6775 9475 6575
+Wire Wire Line
+	9525 6125 9525 6075
+Wire Wire Line
+	9525 6075 9475 6075
+Connection ~ 9650 6125
+Wire Wire Line
+	9325 6325 9325 5975
+Wire Wire Line
+	9325 5975 9850 5975
+Wire Wire Line
+	9850 5975 9850 6025
+Wire Wire Line
+	9850 6025 10050 6025
 $EndSCHEMATC
